Commit message: 更新URDF，完成所有关节和连杆生成

File: mockway_description/urdf/mockway_description.urdf (robot description, URDF)
Before this commit: robot mockway_description, 4 links, 3 joints
Links:
- added link link4, mass 0.371; collision mesh filename=package://mockway_description/meshes/link4.stl; visual mesh filename=package://mockway_description/meshes/link4.stl
- added link link5, mass 0.371; collision mesh filename=package://mockway_description/meshes/link5.stl; visual mesh filename=package://mockway_description/meshes/link5.stl
- added link link6, mass 0.016; collision mesh filename=package://mockway_description/meshes/link6.stl; visual mesh filename=package://mockway_description/meshes/link6.stl
Joints:
- added joint joint4: type revolute, parent link3, child link4, origin xyz=0.000 0.163 0.000 rpy=0.000 -0.000 0.000, axis 0 0 1, limit lower=-6.280 upper=6.280 effort=3.000 velocity=3.140
- added joint joint5: type revolute, parent link4, child link5, origin xyz=0.000 0.000 0.071 rpy=-1.571 0.000 0.000, axis 0 0 1, limit lower=-6.280 upper=6.280 effort=3.000 velocity=3.140
- added joint joint6: type revolute, parent link5, child link6, origin xyz=0.000 -0.039 0.071 rpy=1.571 -0.000 0.000, axis 0 0 1, limit lower=-6.280 upper=6.280 effort=3.000 velocity=3.140
