Commit message: 增加use_mock_hardware参数，用于仿真测试

File: moveit_mockway_config/config/mockway_description.ros2_control.xacro (robot description, xacro)
@@ -1,16 +1,21 @@
 <?xml version="1.0"?>
 <robot xmlns:xacro="http://www.ros.org/wiki/xacro">
-    <xacro:macro name="mockway_description_ros2_control" params="name initial_positions_file">
+    <xacro:macro name="mockway_description_ros2_control" params="name initial_positions_file use_mock_hardware:=false">
         <xacro:property name="initial_positions" value="${xacro.load_yaml(initial_positions_file)['initial_positions']}"/>
         <ros2_control name="${name}" type="system">
             <hardware>
-                <!-- <plugin>mock_components/GenericSystem</plugin> -->
-                <!-- DM Motor Hardware Interface for real hardware -->
-                <plugin>dmmotor_hardware_interface/DMMototHardwareInterface</plugin>
-                <!-- CAN interface configuration -->
-                <!-- <param name="can_interface">can0</param> -->
-                <param name="can_type">usb_can</param>
-                <param name="can_interface">/dev/ttyUSB0</param>
-                <param name="serial_baudrate">921600</param>
+                <xacro:if value="${use_mock_hardware}">
+                    <!-- Mock hardware for simulation / testing -->
+                    <plugin>mock_components/GenericSystem</plugin>
+                </xacro:if>
+                <xacro:unless value="${use_mock_hardware}">
+                    <!-- DM Motor Hardware Interface for real hardware -->
+                    <plugin>dmmotor_hardware_interface/DMMototHardwareInterface</plugin>
+                    <!-- CAN interface configuration -->
+                    <!-- <param name="can_interface">can0</param> -->
+                    <param name="can_type">usb_can</param>
+                    <param name="can_interface">/dev/ttyUSB0</param>
+                    <param name="serial_baudrate">921600</param>
+                </xacro:unless>
             </hardware>
             <!-- Joint 1: DM-J4310-2EC -->

File: moveit_mockway_config/config/mockway_description.urdf.xacro (robot description, xacro)
@@ -2,8 +2,9 @@
 <robot xmlns:xacro="http://www.ros.org/wiki/xacro" name="mockway_description">
     <xacro:arg name="initial_positions_file" default="initial_positions.yaml" />
+    <xacro:arg name="use_mock_hardware" default="false" />
     <!-- Import mockway_description urdf file -->
     <xacro:include filename="$(find mockway_description)/urdf/mockway_description.urdf" />
     <!-- Import control_xacro -->
     <xacro:include filename="mockway_description.ros2_control.xacro" />
-    <xacro:mockway_description_ros2_control name="FakeSystem" initial_positions_file="$(arg initial_positions_file)"/>
+    <xacro:mockway_description_ros2_control name="MockwaySystem" initial_positions_file="$(arg initial_positions_file)" use_mock_hardware="$(arg use_mock_hardware)"/>
 </robot>

Commit message: mac系统moveit模型与通信修复

File: moveit_mockway_config/config/mockway_description.ros2_control.xacro (robot description, xacro)
@@ -1,5 +1,5 @@
 <?xml version="1.0"?>
 <robot xmlns:xacro="http://www.ros.org/wiki/xacro">
-    <xacro:macro name="mockway_description_ros2_control" params="name initial_positions_file use_mock_hardware:=false">
+    <xacro:macro name="mockway_description_ros2_control" params="name initial_positions_file use_mock_hardware:=false can_interface:=/dev/ttyACM0">
         <xacro:property name="initial_positions" value="${xacro.load_yaml(initial_positions_file)['initial_positions']}"/>
         <ros2_control name="${name}" type="system">
@@ -12,7 +12,8 @@
                     <!-- DM Motor Hardware Interface for real hardware -->
                     <plugin>dmmotor_hardware_interface/DMMototHardwareInterface</plugin>
-                    <!-- WSL + 达妙 USB-CAN (2e88:4603) 为 CDC 设备，映射为 /dev/ttyACM0 -->
+                    <!-- 串口设备路径：WSL/Linux 默认 /dev/ttyACM0；macOS 用 /dev/cu.usbmodem* -->
+                    <!-- 可由 launch 参数 can_interface 覆盖，例如 can_interface:=/dev/cu.usbmodem00000000050C1 -->
                     <param name="can_type">usb_can</param>
-                    <param name="can_interface">/dev/ttyACM0</param>
+                    <param name="can_interface">${can_interface}</param>
                     <param name="serial_baudrate">921600</param>
                     <param name="usb_can_adapter">damiao</param>

File: moveit_mockway_config/config/mockway_description.urdf.xacro (robot description, xacro)
@@ -3,8 +3,18 @@
     <xacro:arg name="initial_positions_file" default="initial_positions.yaml" />
     <xacro:arg name="use_mock_hardware" default="false" />
+    <!-- USB-CAN 串口设备：WSL/Linux 默认 /dev/ttyACM0；macOS 传 /dev/cu.usbmodem* -->
+    <xacro:arg name="can_interface" default="/dev/ttyACM0" />
+    <!-- 碰撞几何：mesh(默认, Linux/WSL 用网格) | primitive(macOS 用包围盒, 规避 FCL 在 Eigen5 下崩溃) -->
+    <xacro:arg name="collision_mode" default="mesh" />
+    <xacro:property name="collision_mode_prop" value="$(arg collision_mode)" />
     <!-- Import mockway_description urdf file -->
-    <xacro:include filename="$(find mockway_description)/urdf/mockway_description.urdf" />
+    <xacro:if value="${collision_mode_prop == 'primitive'}">
+        <xacro:include filename="$(find mockway_description)/urdf/mockway_description.primitive_collision.urdf" />
+    </xacro:if>
+    <xacro:unless value="${collision_mode_prop == 'primitive'}">
+        <xacro:include filename="$(find mockway_description)/urdf/mockway_description.urdf" />
+    </xacro:unless>
     <!-- Import control_xacro -->
     <xacro:include filename="mockway_description.ros2_control.xacro" />
-    <xacro:mockway_description_ros2_control name="MockwaySystem" initial_positions_file="$(arg initial_positions_file)" use_mock_hardware="$(arg use_mock_hardware)"/>
+    <xacro:mockway_description_ros2_control name="MockwaySystem" initial_positions_file="$(arg initial_positions_file)" use_mock_hardware="$(arg use_mock_hardware)" can_interface="$(arg can_interface)"/>
 </robot>
